File: motordr.kicad_sch (KiCad schematic)
At the start: 0 parts

Commit message: motor driver ckt
Parts:
- added D1: LED, LED_THT:LED_D3.0mm, symbol Device:LED
- added J1: Conn_01x04_Pin, Connector:FanPinHeader_1x04_P2.54mm_Vertical, symbol Connector:Conn_01x04_Pin
- added J2, J3, J4: Screw_Terminal_01x02, TerminalBlock_Phoenix:TerminalBlock_Phoenix_MKDS-1,5-2-5.08_1x02_P5.08mm_Horizontal, symbol Connector:Screw_Terminal_01x02
- added R1: 1k, Resistor_THT:R_Axial_DIN0204_L3.6mm_D1.6mm_P5.08mm_Horizontal, symbol Device:R
- added U1: L293D, Package_DIP:DIP-16_W7.62mm, symbol Driver_Motor:L293D
- added U3: L7805, Package_TO_SOT_THT:TO-220-3_Vertical, symbol Regulator_Linear:L7805
Connections:
- new net: J3.1 (Pin_1), U1.3 (1Y)
- new net: J3.2 (Pin_2), U1.6 (2Y)
- new net: J2.1 (Pin_1), U1.1 (EN1,2), U1.16 (VCC1), U1.8 (VCC2), U1.9 (EN3,4), U3.1 (IN)
- new net: J1.3 (Pin_3), U1.10 (3A)
- new net: J4.1 (Pin_1), U1.11 (3Y)
- new net: J4.2 (Pin_2), U1.14 (4Y)
- new net: J1.4 (Pin_4), U1.15 (4A)
- new net: J1.1 (Pin_1), U1.2 (1A)
- new net: J1.2 (Pin_2), U1.7 (2A)
- new net: D1.2 (A), R1.2
- new net: R1.1, U3.3 (OUT)
- new net GND: D1.1 (K), J2.2 (Pin_2), U1.12 (GND), U1.13 (GND), U1.4 (GND), U1.5 (GND), U3.2 (GND)
